Commit message: feat: expose chassis/caster dims, add sim-sync helper-per-field hints

File: controller/gogoping-controller/src/vic_pinky/vicpinky_description/urdf/gazebo_control.xacro (robot description, xacro)
@@ -7,6 +7,9 @@
             <left_joint>${prefix}left_wheel_joint</left_joint>
             <right_joint>${prefix}right_wheel_joint</right_joint>
-            <wheel_separation>0.3788</wheel_separation>
-            <wheel_radius>0.0825</wheel_radius>
+            <!-- wheel_separation / wheel_radius 는 robot_core.xacro 에서 YAML
+                 (config/robot_dims.yaml) 로부터 read 한 property 를 재사용 —
+                 single source of truth. -->
+            <wheel_separation>${wheel_separation}</wheel_separation>
+            <wheel_radius>${wheel_radius}</wheel_radius>
             <min_velocity>-1.0</min_velocity>
             <max_velocity>1.0</max_velocity>

File: controller/gogoping-controller/src/vic_pinky/vicpinky_description/urdf/robot_core.xacro (robot description, xacro)
@@ -11,16 +11,14 @@
     <xacro:property name="wheel_x_offset" value="${dims['wheel']['x_offset']}"/>
     <xacro:property name="wheel_z_offset" value="${dims['wheel']['z_offset']}"/>
-    <xacro:property name="chassis_length" value="0.6"/>
-    <xacro:property name="chassis_width" value="0.5"/>
-    <xacro:property name="chassis_height" value="0.128"/>
+    <xacro:property name="chassis_length"   value="${dims['chassis']['length']}"/>
+    <xacro:property name="chassis_width"    value="${dims['chassis']['width']}"/>
+    <xacro:property name="chassis_height"   value="${dims['chassis']['height']}"/>
+    <xacro:property name="chassis_z_offset" value="${dims['chassis']['z_offset']}"/>
     <xacro:property name="chassis_mass" value="50.0"/>
-    <xacro:property name="chassis_z_offset" value="0.087"/>
     <xacro:property name="wheel_mass" value="0.05"/>
-    <xacro:property name="caster_wheel_radius" value="${chassis_z_offset/2}"/>
+    <xacro:property name="caster_wheel_radius" value="${dims['caster']['radius']}"/>
+    <xacro:property name="caster_x_offset"    value="${dims['caster']['x']}"/>
+    <xacro:property name="caster_y_offset"    value="${dims['caster']['y']}"/>
     <xacro:property name="caster_wheel_mass" value="3.0"/>
-    <xacro:property name="caster_x_inset" value="0.056"/>
-    <xacro:property name="caster_y_inset" value="0.156"/>
-    <xacro:property name="caster_x_offset" value="${chassis_length/2 - caster_x_inset}"/>
-    <xacro:property name="caster_y_offset" value="${chassis_width/2 - caster_y_inset}"/>
     <material name="white">
         <color rgba="1 1 1 1" />
