Commit message: refactor: switch robot URDF to v1.0.0 base with 4-pillar frame and update footprint

File: controller/gogoping-controller/src/gogoping/gogoping_navigation/urdf/pinky_kindergarten.urdf.xacro (robot description, xacro)
@@ -1,6 +1,5 @@
 <?xml version="1.0"?>
-<!-- Vic Pinky + 아기자기 유치원 얼굴 데코.
-     vicpinky_description/urdf/robot.urdf.xacro 를 include + visual-only 얼굴 요소 추가.
-     Materials - cute_yellow(머리), cute_white(흰자), cute_black(눈썹/눈동자), cute_red(입/볼). -->
+<!-- Vic Pinky 스폰용 wrapper. vicpinky_description URDF 를 그대로 include.
+     (예전에 유치원 얼굴 데코 link 가 있었으나 사용자 요청으로 제거) -->
 <robot name="pinky" xmlns:xacro="http://www.ros.org/wiki/xacro">
     <xacro:arg name="namespace" default=""/>
@@ -8,120 +7,3 @@
     <!-- 원본 Vic Pinky URDF 로드 -->
     <xacro:include filename="$(find vicpinky_description)/urdf/robot.urdf.xacro"/>
-    <material name="cute_yellow">
-        <color rgba="0.78 0.88 0.20 1"/>
-    </material>
-    <material name="cute_white">
-        <color rgba="1.0 1.0 1.0 1"/>
-    </material>
-    <material name="cute_black">
-        <color rgba="0.05 0.05 0.05 1"/>
-    </material>
-    <material name="cute_red">
-        <color rgba="0.95 0.30 0.30 1"/>
-    </material>
-    <!-- 데코 link - visual 만 모음 -->
-    <link name="${prefix}face_decoration">
-        <inertial>
-            <origin xyz="0 0 0"/>
-            <mass value="0.001"/>
-            <inertia ixx="1e-6" ixy="0" ixz="0" iyy="1e-6" iyz="0" izz="1e-6"/>
-        </inertial>
-        <!-- 1) 노란 머리 박스 (라이다 가리지 않게 앞쪽만 덮음) -->
-        <!--    chassis 앞단 X=0.30, 상단 z=0.064. 머리는 그 앞에 살짝 띄워서. -->
-        <visual name="head_box">
-            <origin xyz="0.305 0 0.10" rpy="0 0 0"/>
-            <geometry>
-                <box size="0.02 0.42 0.26"/>
-            </geometry>
-            <material name="cute_yellow"/>
-        </visual>
-        <!-- 2) 눈 — 흰자 (sphere) -->
-        <visual name="eye_left_white">
-            <origin xyz="0.318 0.10 0.16" rpy="0 0 0"/>
-            <geometry>
-                <sphere radius="0.045"/>
-            </geometry>
-            <material name="cute_white"/>
-        </visual>
-        <visual name="eye_right_white">
-            <origin xyz="0.318 -0.10 0.16" rpy="0 0 0"/>
-            <geometry>
-                <sphere radius="0.045"/>
-            </geometry>
-            <material name="cute_white"/>
-        </visual>
-        <!-- 3) 눈동자 (검은 sphere) -->
-        <visual name="eye_left_pupil">
-            <origin xyz="0.345 0.10 0.16" rpy="0 0 0"/>
-            <geometry>
-                <sphere radius="0.025"/>
-            </geometry>
-            <material name="cute_black"/>
-        </visual>
-        <visual name="eye_right_pupil">
-            <origin xyz="0.345 -0.10 0.16" rpy="0 0 0"/>
-            <geometry>
-                <sphere radius="0.025"/>
-            </geometry>
-            <material name="cute_black"/>
-        </visual>
-        <!-- 4) 눈썹 (검은 box, 눈 위쪽) -->
-        <visual name="brow_left">
-            <origin xyz="0.316 0.10 0.225" rpy="0 0.0 0.20"/>
-            <geometry>
-                <box size="0.005 0.11 0.022"/>
-            </geometry>
-            <material name="cute_black"/>
-        </visual>
-        <visual name="brow_right">
-            <origin xyz="0.316 -0.10 0.225" rpy="0 0.0 -0.20"/>
-            <geometry>
-                <box size="0.005 0.11 0.022"/>
-            </geometry>
-            <material name="cute_black"/>
-        </visual>
-        <!-- 5) 입 (빨간 box, 살짝 곡선 느낌으로 살짝 위쪽 회전) -->
-        <visual name="mouth">
-            <origin xyz="0.316 0 0.05" rpy="0 0 0"/>
-            <geometry>
-                <box size="0.005 0.14 0.025"/>
-            </geometry>
-            <material name="cute_red"/>
-        </visual>
-        <!-- 6) 양쪽 입꼬리 작은 sphere (미소 효과) -->
-        <visual name="smile_left">
-            <origin xyz="0.318 0.075 0.063" rpy="0 0 0"/>
-            <geometry>
-                <sphere radius="0.018"/>
-            </geometry>
-            <material name="cute_red"/>
-        </visual>
-        <visual name="smile_right">
-            <origin xyz="0.318 -0.075 0.063" rpy="0 0 0"/>
-            <geometry>
-                <sphere radius="0.018"/>
-            </geometry>
-            <material name="cute_red"/>
-        </visual>
-        <!-- 7) 작은 볼터치 (분홍 sphere) -->
-        <visual name="cheek_left">
-            <origin xyz="0.316 0.165 0.10" rpy="0 0 0"/>
-            <geometry>
-                <sphere radius="0.025"/>
-            </geometry>
-            <material name="cute_red"/>
-        </visual>
-        <visual name="cheek_right">
-            <origin xyz="0.316 -0.165 0.10" rpy="0 0 0"/>
-            <geometry>
-                <sphere radius="0.025"/>
-            </geometry>
-            <material name="cute_red"/>
-        </visual>
-    </link>
-    <joint name="${prefix}face_decoration_joint" type="fixed">
-        <parent link="${prefix}base_link"/>
-        <child link="${prefix}face_decoration"/>
-        <origin xyz="0 0 0" rpy="0 0 0"/>
-    </joint>
 </robot>

File: controller/gogoping-controller/src/vic_pinky/vicpinky_description/urdf/robot_core.xacro (robot description, xacro)
@@ -1,23 +1,23 @@
 <?xml version="1.0"?>
-<robot name="vicpinky" xmlns:xacro="http://www.ros.org/wiki/xacro">
+<robot name="pinky" xmlns:xacro="http://www.ros.org/wiki/xacro">
     <xacro:arg name="namespace" default=""/>
     <xacro:property name="prefix" value="$(arg namespace)"/>
+    <!-- robot_dims.yaml = single source of truth (urdf-tuner GUI 가 편집).
+         v1.0.0 base + 팀 커스텀 (yaml dim loading + lidar mount/laser yaml 참조). -->
     <xacro:property name="dims_path" value="$(find vicpinky_description)/config/robot_dims.yaml"/>
     <xacro:property name="dims" value="${xacro.load_yaml(dims_path)}"/>
     <xacro:include filename="inertial_macros.xacro"/>
-    <xacro:property name="wheel_radius" value="${dims['wheel']['radius']}"/>
-    <xacro:property name="wheel_thickness" value="${dims['wheel']['thickness']}"/>
     <xacro:property name="wheel_separation" value="${dims['wheel']['separation']}"/>
-    <xacro:property name="wheel_x_offset" value="${dims['wheel']['x_offset']}"/>
-    <xacro:property name="wheel_z_offset" value="${dims['wheel']['z_offset']}"/>
+    <xacro:property name="wheel_radius"     value="${dims['wheel']['radius']}"/>
+    <xacro:property name="wheel_thickness"  value="${dims['wheel']['thickness']}"/>
+    <xacro:property name="wheel_diameter"   value="${2 * wheel_radius}"/>
+    <xacro:property name="wheel_mass" value="0.05"/>
     <xacro:property name="chassis_length"   value="${dims['chassis']['length']}"/>
     <xacro:property name="chassis_width"    value="${dims['chassis']['width']}"/>
     <xacro:property name="chassis_height"   value="${dims['chassis']['height']}"/>
-    <xacro:property name="chassis_z_offset" value="${dims['chassis']['z_offset']}"/>
-    <xacro:property name="chassis_mass" value="50.0"/>
-    <xacro:property name="wheel_mass" value="0.05"/>
+    <xacro:property name="chassis_mass"     value="50.0"/>
+    <!-- chassis 가 base_link (휠축) 기준 어디 centered 인가. v1.0.0: -length/2+0.1 = -0.2 -->
+    <xacro:property name="chassis_x_offset" value="${-chassis_length/2 + 0.1}"/>
     <xacro:property name="caster_wheel_radius" value="${dims['caster']['radius']}"/>
-    <xacro:property name="caster_x_offset"    value="${dims['caster']['x']}"/>
-    <xacro:property name="caster_y_offset"    value="${dims['caster']['y']}"/>
     <xacro:property name="caster_wheel_mass" value="3.0"/>
     <material name="white">
@@ -33,20 +33,63 @@
         <color rgba="0 0 1 1"/>
     </material>
+    <!-- v1.0.0 의 4-pillar + top plate 구조 (placeholder 박스로 시각 확보) -->
+    <xacro:property name="pillar_mass" value="0.1"/>
+    <xacro:property name="pillar_size" value="0.03"/>
+    <xacro:property name="pillar_height" value="0.5"/>
+    <xacro:property name="pillar_inset" value="0.015"/>
+    <xacro:macro name="pillar" params="prefix x y">
+        <visual>
+            <origin xyz="${x} ${y} ${chassis_height + pillar_height/2 - 0.02}" rpy="0 0 0"/>
+            <geometry>
+                <box size="${pillar_size} ${pillar_size} ${pillar_height}"/>
+            </geometry>
+            <material name="gray"/>
+        </visual>
+        <collision>
+            <origin xyz="${x} ${y} ${chassis_height + pillar_height/2 - 0.02}" rpy="0 0 0"/>
+            <geometry>
+                <box size="${pillar_size} ${pillar_size} ${pillar_height}"/>
+            </geometry>
+        </collision>
+        <xacro:inertial_box mass="${pillar_mass}" x="${pillar_size}" y="${pillar_size}" z="${pillar_height}">
+            <origin xyz="${x} ${y} ${chassis_height + pillar_height/2 - 0.02}" rpy="0 0 0"/>
+        </xacro:inertial_box>
+    </xacro:macro>
     <link name="${prefix}base_link">
         <visual>
-            <origin xyz="0 0 0" rpy="0 0 0"/>
-            <geometry>
-                <mesh filename="package://vicpinky_description/meshes/visual/base_link.stl" scale="1 1 1"/>
-            </geometry>
-            <material name="gray"/>
-        </visual>
-        <collision>
-            <origin xyz="0 0 ${chassis_height/2-0.02}" rpy="0 0 0"/>
+            <origin xyz="${chassis_x_offset} 0 ${chassis_height/2-0.02}" rpy="0 0 0"/>
             <geometry>
                 <box size="${chassis_length} ${chassis_width} ${chassis_height}"/>
             </geometry>
+            <material name="gray"/>
+        </visual>
+        <collision>
+            <origin xyz="${chassis_x_offset} 0 ${chassis_height/2-0.02}" rpy="0 0 0"/>
+            <geometry>
+                <box size="${chassis_length} ${chassis_width} ${chassis_height}"/>
+            </geometry>
         </collision>
         <xacro:inertial_box mass="${chassis_mass}" x="${chassis_length}" y="${chassis_width}" z="${chassis_height}">
             <origin xyz="0 0 0" rpy="0 0 0"/>
+        </xacro:inertial_box>
+        <xacro:pillar prefix="front_left"  x="${chassis_x_offset + chassis_length/2 - pillar_inset}" y="${chassis_width/2 - pillar_inset}"/>
+        <xacro:pillar prefix="front_right" x="${chassis_x_offset + chassis_length/2 - pillar_inset}" y="-${chassis_width/2 - pillar_inset}"/>
+        <xacro:pillar prefix="rear_left"   x="${chassis_x_offset - chassis_length/2 + pillar_inset}" y="${chassis_width/2 - pillar_inset}"/>
+        <xacro:pillar prefix="rear_right"  x="${chassis_x_offset - chassis_length/2 + pillar_inset}" y="-${chassis_width/2 - pillar_inset}"/>
+        <visual>
+            <origin xyz="${chassis_x_offset} 0 ${chassis_height/2 + pillar_height + 0.03}" rpy="0 0 0"/>
+            <geometry>
+                <box size="${chassis_length} ${chassis_width} 0.03"/>
+            </geometry>
+            <material name="gray"/>
+        </visual>
+        <collision>
+            <origin xyz="${chassis_x_offset} 0 ${chassis_height/2 + pillar_height + 0.03}" rpy="0 0 0"/>
+            <geometry>
+                <box size="${chassis_length} ${chassis_width} 0.03"/>
+            </geometry>
+        </collision>
+        <xacro:inertial_box mass="${chassis_mass}" x="${chassis_length}" y="${chassis_width}" z="0.03">
+            <origin xyz="${chassis_x_offset} 0 ${chassis_height/2 + pillar_height + 0.03}" rpy="0 0 0"/>
         </xacro:inertial_box>
     </link>
@@ -55,17 +98,17 @@
         <parent link="${prefix}base_footprint"/>
         <child link="${prefix}base_link"/>
-        <origin xyz="0 0 ${chassis_z_offset}" rpy="0 0 0"/>
+        <origin xyz="0 0 ${wheel_diameter/2}" rpy="0 0 0"/>
     </joint>
     <joint name="${prefix}left_wheel_joint" type="continuous">
         <parent link="${prefix}base_link"/>
         <child link="${prefix}left_wheel"/>
-        <origin xyz="${wheel_x_offset} ${wheel_separation/2} ${wheel_z_offset}" rpy="-${pi/2} 0 0"/>
+        <origin xyz="0 ${wheel_separation/2} 0" rpy="-${pi/2} 0 0"/>
         <axis xyz="0 0 1"/>
     </joint>
     <link name="${prefix}left_wheel">
         <visual>
-            <origin xyz="0 0 0" rpy="0 ${-pi/2} 0"/>
-            <geometry>
-                <mesh filename="package://vicpinky_description/meshes/visual/wheel.stl" scale="1 1 1"/>
+            <origin xyz="0 0 0" rpy="0 0 0"/>
+            <geometry>
+                <cylinder radius="${wheel_radius}" length="${wheel_thickness}"/>
             </geometry>
             <material name="black"/>
@@ -84,12 +127,12 @@
         <parent link="${prefix}base_link"/>
         <child link="${prefix}right_wheel"/>
-        <origin xyz="${wheel_x_offset} ${-1 * wheel_separation/2} ${wheel_z_offset}" rpy="${pi/2} 0 0"/>
+        <origin xyz="0 ${-1 * wheel_separation/2} 0" rpy="${pi/2} 0 0"/>
         <axis xyz="0 0 -1"/>
     </joint>
     <link name="${prefix}right_wheel">
         <visual>
-            <origin xyz="0 0.0 0.0" rpy="0 ${-pi/2} 0"/>
-            <geometry>
-                <mesh filename="package://vicpinky_description/meshes/visual/wheel.stl" scale="1 1 1"/>
+            <origin xyz="0 0 0" rpy="0 0 0"/>
+            <geometry>
+                <cylinder radius="${wheel_radius}" length="${wheel_thickness}"/>
             </geometry>
             <material name="black"/>
@@ -105,33 +148,50 @@
         </xacro:inertial_cylinder>
     </link>
-    <xacro:macro name="caster_wheel" params="suffix x_offset y_offset">
-        <joint name="${prefix}${suffix}_caster_joint" type="fixed">
-            <parent link="${prefix}base_link"/>
-            <child link="${prefix}${suffix}_caster"/>
-            <origin xyz="${x_offset} ${y_offset} ${-chassis_z_offset + caster_wheel_radius}" rpy="0 0 0"/>
-        </joint>
-        <link name="${prefix}${suffix}_caster">
-            <visual>
-                <origin xyz="0 0 ${caster_wheel_radius}" rpy="0 0 0"/>
-                <geometry>
-                    <mesh filename="package://vicpinky_description/meshes/visual/caster.stl" scale="1 1 1"/>
-                </geometry>
-                <material name="gray"/>
-            </visual>
-            <collision>
-                <origin xyz="0 0 0" rpy="0 0 0"/>
-                <geometry>
-                    <sphere radius="${caster_wheel_radius}"/>
-                </geometry>
-            </collision>
-            <xacro:inertial_sphere mass="${caster_wheel_mass}" radius="${caster_wheel_radius}">
-                <origin xyz="0 0 0" rpy="0 0 0"/>
-            </xacro:inertial_sphere>
-        </link>
-    </xacro:macro>
-    <xacro:caster_wheel suffix="front_left"  x_offset="${caster_x_offset}"  y_offset="${caster_y_offset}"/>
-    <xacro:caster_wheel suffix="front_right" x_offset="${caster_x_offset}"  y_offset="${-caster_y_offset}"/>
-    <xacro:caster_wheel suffix="rear_left"   x_offset="${-caster_x_offset}" y_offset="${caster_y_offset}"/>
-    <xacro:caster_wheel suffix="rear_right"  x_offset="${-caster_x_offset}" y_offset="${-caster_y_offset}"/>
+    <joint name="${prefix}left_caster_joint" type="fixed">
+        <parent link="${prefix}base_link"/>
+        <child link="${prefix}left_caster"/>
+        <origin xyz="${-chassis_length/2-0.1} ${chassis_width/2-0.1} ${-2*caster_wheel_radius+0.015}" rpy="0 0 0"/>
+    </joint>
+    <link name="${prefix}left_caster">
+        <visual>
+            <origin xyz="0 0 0" rpy="0 0 0"/>
+            <geometry>
+                <sphere radius="${caster_wheel_radius}"/>
+            </geometry>
+            <material name="gray"/>
+        </visual>
+        <collision>
+            <origin xyz="0 0 0" rpy="0 0 0"/>
+            <geometry>
+                <sphere radius="${caster_wheel_radius}"/>
+            </geometry>
+        </collision>
+        <xacro:inertial_sphere mass="${caster_wheel_mass}" radius="${caster_wheel_radius}">
+            <origin xyz="0 0 0" rpy="0 0 0"/>
+        </xacro:inertial_sphere>
+    </link>
+    <joint name="${prefix}right_caster_joint" type="fixed">
+        <parent link="${prefix}base_link"/>
+        <child link="${prefix}right_caster"/>
+        <origin xyz="${-chassis_length/2-0.1} ${-chassis_width/2+0.1} ${-2*caster_wheel_radius+0.015}" rpy="0 0 0"/>
+    </joint>
+    <link name="${prefix}right_caster">
+        <visual>
+            <origin xyz="0 0 0" rpy="0 0 0"/>
+            <geometry>
+                <sphere radius="${caster_wheel_radius}"/>
+            </geometry>
+            <material name="gray"/>
+        </visual>
+        <collision>
+            <origin xyz="0 0 0" rpy="0 0 0"/>
+            <geometry>
+                <sphere radius="${caster_wheel_radius}"/>
+            </geometry>
+        </collision>
+        <xacro:inertial_sphere mass="${caster_wheel_mass}" radius="${caster_wheel_radius}">
+            <origin xyz="0 0 0" rpy="0 0 0"/>
+        </xacro:inertial_sphere>
+    </link>
     <link name="${prefix}lidar_mount">
         <visual>
@@ -140,4 +200,5 @@
                 <mesh filename="package://vicpinky_description/meshes/visual/lidar.dae" scale="1 1 1"/>
             </geometry>
+            <material name="blue"/>
         </visual>
         <collision>
@@ -152,4 +213,20 @@
             <inertia ixx="0.000058" ixy="0" ixz="0.000005" iyy="0.000099" iyz="0" izz="0.000103"/>
         </inertial>
+        <visual>
+            <origin xyz="0 0 -0.035" rpy="0 0 0"/>
+            <geometry>
+                <box size="0.07 0.07 0.07"/>
+            </geometry>
+            <material name="blue"/>
+        </visual>
+        <collision>
+            <origin xyz="0 0 -0.035" rpy="0 0 0"/>
+            <geometry>
+                <box size="0.07 0.07 0.07"/>
+            </geometry>
+        </collision>
+        <xacro:inertial_box mass="0.03" x="0.07" y="0.07" z="0.07">
+            <origin xyz="0 0 -0.035" rpy="0 0 0"/>
+        </xacro:inertial_box>
     </link>
     <joint name="${prefix}lidar_mount_fixed_joint" type="fixed">
