Commit message: feat(eduping): 뎁스카메라 뷰 통합 + octomap/servo 인프라
4b98dc6 가 추가했지만 미연결로 남아있던 wiring 들을 한꺼번에 잇고,
Phase 1-4 (octomap → servo → twist driver) 인프라를 도입.

depth 파이프라인 마무리:
- streaming/app.py 에 depth_ws_router include — 이전엔 producer WS 가 HTTP 403
- vite.config.ts 에 /ws/depth-stream proxy rule
- App.vue 에 DepthViewer 마운트 + '뎁스카메라 뷰' mode (shared/robots.json)
- OpenarmViewer 에 useDepthCloudInScene 연결 + showFrustum=true 명시
- useHandTracker — initialize() 명시 호출 + ready flag 로 loading UX 수정
- public/urdf/openarm_v10/openarm.urdf 재생성 (D435 link 추가, mount z=0.62)
- public/urdf/openarm_v10/regenerate.sh helper

highfive 동적 IK reach:
- /api/eduping/highfive/hand-target POST → ROS PointStamped publisher
- highfive_node 의 avoid_collisions 는 sim 의 빈 planning scene + 보수적 SRDF
  로 KDL 이 IK 전부 reject 해서 일단 False (TRAC-IK 또는 planning scene 통합 후 True)

Phase 1+2 — D435 → octomap planning scene:
- eduarm/config/sensors_3d.yaml — DepthImageOctomapUpdater (≤4cm 근접 기준)
- eduarm/launch/d435_camera.launch.py — realsense2_camera wrapper
- eduarm/launch/octomap_demo[_sim].launch.py — 실/sim 데모
- eduarm/rviz/octomap.rviz — RViz preset

Phase 3 — MoveIt Servo (collision-aware halt):
- eduarm/config/servo.yaml — check_collisions=true, scene/self proximity
- eduarm/launch/servo.launch.py — arm:=left|right 파라미터화

Phase 4 — TwistStamped driver:
- eduarm/eduarm/servo_reach_node.py — PointStamped → cartesian P → twist
- package.xml + setup.py 갱신 (moveit_servo, geometry_msgs, tf2_*; 누락된
  d435_depth_streamer / highfive_node entry_point 추가)

File: service/web-service/robot-web/public/urdf/openarm_v10/openarm.urdf (robot description, URDF)
Before this commit: robot openarm, 26 links, 25 joints
Links:
- added link d435_depth_optical_frame
- added link d435_link, mass 0.07; collision box size=0.025 0.09 0.025; visual box size=0.025 0.09 0.025
Joints:
- added joint d435_depth_optical_joint: type fixed, parent d435_link, child d435_depth_optical_frame, origin xyz=0 0 0 rpy=-1.5708 0 -1.5708
- added joint d435_mount_joint: type fixed, parent openarm_body_link0, child d435_link, origin xyz=0.05 0.0 0.62 rpy=0 0 0

Commit message: feat(doctor): leader_passthrough 고정주기 출력 + EMA + 방향성 장애물 차단
WS 도착(버스트)과 출력을 분리 — 고정주기 타이머가 EMA 저역통과 + 속도 캡으로
publish 해 도착 지터발 떨림 제거. d435 voxel(/eduping/world_voxels)로 forearm
(link4)-장애물 최근접 거리를 계산, block_dist 내 진입 시 안전자세 쪽 성분만 허용
(전진 차단·후퇴 허용), release_dist 회복 시 해제(히스테리시스). voxel/TF 누락 시
fail-open. device-eduping.sh 에 튜닝 파라미터 노출, urdf d435 마운트 위치 보정.

File: service/web-service/robot-web/public/urdf/openarm_v10/openarm.urdf (robot description, URDF)
Before this commit: robot openarm, 28 links, 27 joints
Joints:
- joint d435_mount_joint: origin xyz=0.05 0.0 0.62 rpy=0 0 0 -> xyz=0.075 0.0 0.68 rpy=0 0 0
